File: Version 1.0/Circuit Board/Aegis PCB - 1 v113.brd (EAGLE design)
At the start: 94.1 x 108.1 mm, 99 parts

Commit message: Adding updated circuit boards and gerber files
Parts:
- removed R10, R8, R9: 10K, Personal:RES-603
- added TP10, TP11, TP12, TP13, TP15, TP4, TP5, TP7, TP8: TESTPOINT, Personal:TESTPOINT
- moved R18 6.82 mm to (25.7, 31.9), turned to 90 degrees
- moved TP2 1.32 mm to (18.2, 47.1)
- moved SD1 0.35 mm to (47.9, 58.6)
- moved TP3 0.27 mm to (13.8, 47.1)
- moved R4 0.12 mm to (36.8, 28.7)
- renumbered U$9 to RASPBERRY_PI_CM4
Connections:
- new net RP_RX: BOARD_CONN1.16, RASPBERRY_PI_CM4.51
- new net RP_TX: BOARD_CONN1.17, RASPBERRY_PI_CM4.55
- net BAT: now also TP4.TP
- net BUT_PWR: now also TP8.TP
- net DCDC_EN: now also TP11.TP; no longer R8.A
- net GAUGE_ALERT: now also RASPBERRY_PI_CM4.45
- net GND: no longer BOARD_CONN1.18, R10.C, R8.C, R9.C
- net INT: now also RASPBERRY_PI_CM4.41
- net LCD_EN: now also TP15.TP; no longer R10.A
- net LCD_RST: now also TP13.TP
- net LCD_RST_ADJ: now also TP12.TP; no longer R9.A
- net PWR_EN: now also TP10.TP
- net VBUS1: now also BOARD_CONN1.18; no longer BOARD_CONN1.16, BOARD_CONN1.17
- net VREF3.3: now also TP7.TP
- net VREF5.0: now also TP5.TP
Routing:
- net INT: track 3.95 -> 60.3 mm, vias 0 -> 2
- net GAUGE_ALERT: track 27.2 -> 79.6 mm, vias 4 -> 3
- net RP_RX: track 0.00 -> 37.8 mm, vias 0 -> 2
- net RP_TX: track 0.00 -> 37.3 mm, vias 0 -> 2
- net HDMI0_D1_P: track 127.9 -> 131.0 mm
- net HDMI0_D1_N: track 127.9 -> 131.0 mm
- net HDMI0_CK_N: track 127.9 -> 131.0 mm
- net HDMI0_CK_P: track 127.9 -> 131.0 mm
- net HDMI0_D0_N: track 127.9 -> 131.0 mm
- net HDMI0_D2_N: track 127.9 -> 131.0 mm
- net HDMI0_D0_P: track 127.9 -> 131.0 mm
- net HDMI0_D2_P: track 127.9 -> 131.0 mm
- net SCL1: track 117.7 -> 114.9 mm, vias 8 -> 6
- net SDA1: track 117.7 -> 114.9 mm, vias 8 -> 6
- net RP1.8: track 42.9 -> 45.5 mm
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- removed copper zone on layer 1, net VBUS1
Other:
- outline, holes or cut-outs redrawn
