File: Version 1.0/Circuit Board/Aegis PCB - 1 v58.sch (EAGLE design)
At the start: 99 parts

Commit message: Adding updated circuit boards and gerber files
Parts:
- removed R10, R8, R9: 10K, Personal:RES-603
- added TP10, TP11, TP12, TP13, TP15, TP4, TP5, TP7, TP8: TESTPOINT, Personal:TESTPOINT
- renumbered U$9 to RASPBERRY_PI_CM4
Connections:
- new net RP_RX: BOARD_CONN1.16, RASPBERRY_PI_CM4.51
- new net RP_TX: BOARD_CONN1.17, RASPBERRY_PI_CM4.55
- net BAT: now also TP4.TP
- net BUT_PWR: now also TP8.TP
- net DCDC_EN: now also TP11.TP; no longer R8.A
- net GAUGE_ALERT: now also RASPBERRY_PI_CM4.45
- net GND: no longer BOARD_CONN1.18, R10.C, R8.C, R9.C
- net INT: now also RASPBERRY_PI_CM4.41
- net LCD_EN: now also TP15.TP; no longer R10.A
- net LCD_RST: now also TP13.TP
- net LCD_RST_ADJ: now also TP12.TP; no longer R9.A
- net PWR_EN: now also TP10.TP
- net VBUS1: now also BOARD_CONN1.18; no longer BOARD_CONN1.16, BOARD_CONN1.17
- net VREF3.3: now also TP7.TP
- net VREF5.0: now also TP5.TP
